File: Numpad.sch (KiCad schematic (older format))
At the start: 50 parts, among them SW1 SW_Push, U1 ATmega32U4-AU, Y1 16MHz

Commit message: Commit all files before starting from scratch
Parts:
- U: renamed from U1; value ATmega32U4-AU -> ATmega32U4-MU; footprint Package_QFP:TQFP-44_10x10mm_P0.8mm -> Package_DFN_QFN:QFN-44-1EP_7x7mm_P0.5mm_EP5.2x5.2mm; symbol MCU_Microchip_ATmega:ATmega32U4-AU -> MCU_Microchip_ATmega:ATmega32U4-MU
Connections:
- net labels added: USB_D+, USB_D-
- no-connect marks 19 -> 20
Other:
- moved on the sheet: F1, R2, R3
Changed lines of the file:
@@
 L Device:R_Small R2
 U 1 1 5F46DCA0
-P 4500 2900
-F 0 "R2" V 4430 2900 50  0000 C CNN
-F 1 "22" V 4500 2900 50  0000 C CNN
-F 2 "Resistor_SMD:R_0805_2012Metric" H 4500 2900 50  0001 C CNN
-F 3 "~" H 4500 2900 50  0001 C CNN
-	1    4500 2900
+P 4300 2900
+F 0 "R2" V 4230 2900 50  0000 C CNN
+F 1 "22" V 4300 2900 50  0000 C CNN
+F 2 "Resistor_SMD:R_0805_2012Metric" H 4300 2900 50  0001 C CNN
+F 3 "~" H 4300 2900 50  0001 C CNN
+	1    4300 2900
 	0    1    1    0
 $EndComp
@@
 L Device:R_Small R3
 U 1 1 5F46E5A5
-P 4500 3000
-F 0 "R3" V 4570 3000 50  0000 C CNN
-F 1 "22" V 4500 3000 50  0000 C CNN
-F 2 "Resistor_SMD:R_0805_2012Metric" H 4500 3000 50  0001 C CNN
-F 3 "~" H 4500 3000 50  0001 C CNN
-	1    4500 3000
+P 4300 3000
+F 0 "R3" V 4370 3000 50  0000 C CNN
+F 1 "22" V 4300 3000 50  0000 C CNN
+F 2 "Resistor_SMD:R_0805_2012Metric" H 4300 3000 50  0001 C CNN
+F 3 "~" H 4300 3000 50  0001 C CNN
+	1    4300 3000
 	0    1    1    0
 $EndComp
@@
 	1    0    0    -1
 $EndComp
-Text GLabel 4250 2900 0    50   Input ~ 0
+Text GLabel 4050 2900 0    50   Input ~ 0
 D+
-Text GLabel 4250 3000 0    50   Input ~ 0
+Text GLabel 4050 3000 0    50   Input ~ 0
 D-
 $Comp
@@
 L Device:Polyfuse_Small F1
 U 1 1 5F49EC26
-P 2450 1550
-F 0 "F1" V 2245 1550 50  0000 C CNN
-F 1 "500mA" V 2336 1550 50  0000 C CNN
-F 2 "Fuse:Fuse_1206_3216Metric" H 2500 1350 50  0001 L CNN
-F 3 "~" H 2450 1550 50  0001 C CNN
-	1    2450 1550
+P 2450 1650
+F 0 "F1" V 2245 1650 50  0000 C CNN
+F 1 "500mA" V 2336 1650 50  0000 C CNN
+F 2 "Fuse:Fuse_1206_3216Metric" H 2500 1450 50  0001 L CNN
+F 3 "~" H 2450 1650 50  0001 C CNN
+	1    2450 1650
 	0    1    1    0
 $EndComp
@@
 L power:VCC #PWR01
 U 1 1 5F4A46A3
-P 2250 1450
-F 0 "#PWR01" H 2250 1300 50  0001 C CNN
-F 1 "VCC" H 2267 1623 50  0000 C CNN
-F 2 "" H 2250 1450 50  0001 C CNN
-F 3 "" H 2250 1450 50  0001 C CNN
-	1    2250 1450
+P 2250 1550
+F 0 "#PWR01" H 2250 1400 50  0001 C CNN
+F 1 "VCC" H 2267 1723 50  0000 C CNN
+F 2 "" H 2250 1550 50  0001 C CNN
+F 3 "" H 2250 1550 50  0001 C CNN
+	1    2250 1550
 	1    0    0    -1
 $EndComp
@@
 L power:+5V #PWR02
 U 1 1 5F4A5296
-P 2650 1450
-F 0 "#PWR02" H 2650 1300 50  0001 C CNN
-F 1 "+5V" H 2665 1623 50  0000 C CNN
-F 2 "" H 2650 1450 50  0001 C CNN
-F 3 "" H 2650 1450 50  0001 C CNN
-	1    2650 1450
+P 2650 1550
+F 0 "#PWR02" H 2650 1400 50  0001 C CNN
+F 1 "+5V" H 2665 1723 50  0000 C CNN
+F 2 "" H 2650 1550 50  0001 C CNN
+F 3 "" H 2650 1550 50  0001 C CNN
+	1    2650 1550
 	1    0    0    -1
 $EndComp
@@
 ROW4
 $Comp
-L MCU_Microchip_ATmega:ATmega32U4-AU U1
+L MCU_Microchip_ATmega:ATmega32U4-MU U
 U 1 1 5F4609DF
 P 5400 3400
-F 0 "U1" V 4750 1800 50  0000 C CNN
-F 1 "ATmega32U4-AU" V 4850 2050 50  0000 C CNN
-F 2 "Package_QFP:TQFP-44_10x10mm_P0.8mm" H 5400 3400 50  0001 C CIN
+F 0 "U" V 4750 1800 50  0000 C CNN
+F 1 "ATmega32U4-MU" V 4850 2050 50  0000 C CNN
+F 2 "Package_DFN_QFN:QFN-44-1EP_7x7mm_P0.5mm_EP5.2x5.2mm" H 5400 3400 50  0001 C CIN
 F 3 "http://ww1.microchip.com/downloads/en/DeviceDoc/Atmel-7766-8-bit-AVR-ATmega16U4-32U4_Datasheet.pdf" H 5400 3400 50  0001 C CNN
 	1    5400 3400
@@
 $EndComp
 Wire Wire Line
-	4600 2900 4800 2900
-Wire Wire Line
-	4800 3000 4600 3000
-Wire Wire Line
-	4400 3000 4250 3000
-Wire Wire Line
-	4400 2900 4250 2900
+	4200 3000 4050 3000
+Wire Wire Line
+	4200 2900 4050 2900
 Wire Wire Line
 	4600 3650 4600 3500
@@
 	2100 2050 2100 2100
 Wire Wire Line
-	1950 1550 2250 1550
-Wire Wire Line
-	2550 1550 2650 1550
-Wire Wire Line
-	2650 1550 2650 1450
-Wire Wire Line
-	2250 1450 2250 1550
-Connection ~ 2250 1550
-Wire Wire Line
-	2250 1550 2350 1550
+	1950 1650 2250 1650
+Wire Wire Line
+	2550 1650 2650 1650
+Wire Wire Line
+	2650 1650 2650 1550
+Wire Wire Line
+	2250 1550 2250 1650
+Connection ~ 2250 1650
+Wire Wire Line
+	2250 1650 2350 1650
 Wire Notes Line
 	1000 2350 1000 1000
@@
 	1000 4100 3000 4100
 Wire Notes Line
-	3000 1000 3000 2350
+	2800 1000 2800 2350
 Wire Notes Line
 	1000 2350 3000 2350
@@
 $EndComp
 NoConn ~ 4800 2500
-NoConn ~ 1950 1650
 NoConn ~ 1950 1950
 NoConn ~ 6000 4800
@@
 NoConn ~ 6000 1900
 NoConn ~ 6000 4100
+NoConn ~ 1950 1550
+NoConn ~ 10800 2250
+Text Label 4450 2900 0    50   ~ 0
+USB_D+
+Wire Wire Line
+	4400 2900 4800 2900
+Wire Wire Line
+	4400 3000 4800 3000
+Text Label 4450 3000 0    50   ~ 0
+USB_D-
 $EndSCHEMATC

Commit message: Restart project
Parts:
- removed C7: 1uF, Capacitor_SMD:C_1206_3216Metric, symbol Device:C_Small
- removed D1, D10, D11, D12, D13, D14, D15, D16, D17, D2, D3, D4, D5, D6, D7, D8, D9: D_Small, Diode_SMD:D_SOD-123, symbol Device:D_Small
- removed MX14, MX17, MX4, MX5, MX6, MX7, MX9: MX-NoLED, MX_Alps_Hybrid:MX-1U-NoLED, symbol MX_Alps_Hybrid:MX-NoLED
- removed MX15, MX8: MX-NoLED, MX_Alps_Hybrid:MX-2U-ReversedStabilizers-Vertical-NoLED, symbol MX_Alps_Hybrid:MX-NoLED
- removed MX16: MX-NoLED, MX_Alps_Hybrid:MX-2U-ReversedStabilizers-NoLED, symbol MX_Alps_Hybrid:MX-NoLED
- removed U: ATmega32U4-MU, Package_DFN_QFN:QFN-44-1EP_7x7mm_P0.5mm_EP5.2x5.2mm, symbol MCU_Microchip_ATmega:ATmega32U4-MU
- removed USB1: Molex-0548190589, random-keyboard-parts:Molex-0548190589, symbol random-keyboard-parts:Molex-0548190589
- removed Y1: 16MHz, Crystal:Crystal_SMD_3225-4Pin_3.2x2.5mm, symbol Device:Crystal_GND24_Small
- added D0, D1, D10, D11, D12, D13, D2, D20, D21, D22, D3, D30, D31, D32, D33, D40, D42: D_Small_ALT, Diode_SMD:D_SOD-123, symbol Device:D_Small_ALT
- added MX0, MX20, MX21, MX22, MX30, MX31, MX32, MX42: MX-NoLED, MX_Only:MXOnly-1U-NoLED, symbol MX_Alps_Hybrid:MX-NoLED
- added MX33, MX40: MX-NoLED, MX_Only:MXOnly-2U-ReversedStabilizers-NoLED, symbol MX_Alps_Hybrid:MX-NoLED
- added R5: 22R, Resistor_SMD:R_0402_1005Metric, symbol Device:R_Small
- added R6: 10k, Resistor_SMD:R_0402_1005Metric, symbol Device:R_Small
- added U1: USBLC6-2SC6, Package_TO_SOT_SMD:SOT-23-6, symbol Power_Protection:USBLC6-2SC6
- added U2: ATmega32U2-MU, Package_DFN_QFN:QFN-32-1EP_5x5mm_P0.5mm_EP3.1x3.1mm, symbol MCU_Microchip_ATmega:ATmega32U2-MU
- added USB1: HRO-TYPE-C-31-M-12, Type-C:HRO-TYPE-C-31-M-12, symbol Type-C:HRO-TYPE-C-31-M-12
- added Y1: 16MHz, Crystal:Crystal_SMD_3225-4Pin_3.2x2.5mm, symbol Device:Crystal_GND24
- C1, C2: value 22pF -> 100nF; footprint Capacitor_SMD:C_1206_3216Metric -> Capacitor_SMD:C_0402_1005Metric; LCSC (none) -> C1525
- C3: value 0.1uF -> 10uF; footprint Capacitor_SMD:C_1206_3216Metric -> Capacitor_SMD:C_0603_1608Metric; LCSC (none) -> C19702
- C4, C5: value 0.1uF -> 22pF; footprint Capacitor_SMD:C_1206_3216Metric -> Capacitor_SMD:C_0402_1005Metric; LCSC (none) -> C1555
- C6: value 10uF -> 1uF; footprint Capacitor_SMD:C_1206_3216Metric -> Capacitor_SMD:C_0402_1005Metric; LCSC (none) -> C52923
- F1: footprint Fuse:Fuse_1206_3216Metric -> Fuse:Fuse_0603_1608Metric; LCSC (none) -> C261937
- MX1, MX10, MX11, MX12, MX2, MX3: footprint MX_Alps_Hybrid:MX-1U-NoLED -> MX_Only:MXOnly-1U-NoLED
- MX13: footprint MX_Alps_Hybrid:MX-1U-NoLED -> MX_Only:MXOnly-2U-ReversedStabilizers-NoLED
- R1: value 10k -> 5.1k; footprint Resistor_SMD:R_0805_2012Metric -> Resistor_SMD:R_0402_1005Metric; LCSC (none) -> C25905
- R2: value 22 -> 5.1k; footprint Resistor_SMD:R_0805_2012Metric -> Resistor_SMD:R_0402_1005Metric; LCSC (none) -> C25905
- R3: value 22 -> 10k; footprint Resistor_SMD:R_0805_2012Metric -> Resistor_SMD:R_0402_1005Metric; LCSC (none) -> C25744
- R4: value 10k -> 22R; footprint Resistor_SMD:R_0805_2012Metric -> Resistor_SMD:R_0402_1005Metric; LCSC (none) -> C25092
- SW1: footprint random-keyboard-parts:SKQG-1155865 -> Switches:TACTILE_SWITCH_SMD_5.2MM; LCSC (none) -> C318884
Connections:
- net +5V: now also C1.1, C2.1, R3.1, U1.5 (VBUS), U2.31 (UVCC), U2.32 (AVCC), U2.4 (VCC); no longer C4.1, C5.1, C6.1, R1.1
- net COL0: now also MX10.1 (COL), MX0.1 (COL), MX20.1 (COL), MX30.1 (COL), MX40.1 (COL), U2.23 (PC6); no longer MX1.1 (COL), MX12.1 (COL)
- net COL1: now also MX1.1 (COL), MX11.1 (COL), MX21.1 (COL), MX31.1 (COL), U2.11 (PD5); no longer MX10.1 (COL), MX13.1 (COL), MX2.1 (COL)
- net COL2: now also MX12.1 (COL), MX2.1 (COL), MX22.1 (COL), MX32.1 (COL), MX42.1 (COL), U2.10 (PD4); no longer MX11.1 (COL), MX3.1 (COL)
- net COL3: now also MX13.1 (COL), MX3.1 (COL), MX33.1 (COL), U2.9 (PD3)
- net D+: now also R4.2, U1.3 (IO2); no longer R2.2
- net D-: now also R5.2, U1.1 (IO1); no longer R3.2
- net GND: now also C1.2, R1.2, R2.2, R6.1, U1.2 (GND), U2.28 (UGND), U2.3 (GND), U2.33 (GND), USB1.1 (GND), USB1.12 (GND), Y1.2, Y1.4; no longer C1.1, R4.1
- net ROW0: now also D0.1 (K), D1.1 (K), D2.1 (K), D3.1 (K), U2.25 (PC5)
- net ROW1: now also D10.1 (K), D11.1 (K), D12.1 (K), D13.1 (K), U2.17 (PB3)
- net ROW2: now also D20.1 (K), D21.1 (K), D22.1 (K), U2.16 (PB2)
- net ROW3: now also D30.1 (K), D31.1 (K), D32.1 (K), D33.1 (K), U2.15 (PB1)
- net ROW4: now also D40.1 (K), D42.1 (K), U2.14 (PB0)
- net USB_D+: now also U1.4 (IO2), USB1.6 (DP1), USB1.8 (DP2); no longer R2.1
- net USB_D-: now also U1.6 (IO1), USB1.5 (DN2), USB1.7 (DN1); no longer R3.1
- net VCC: now also USB1.11 (VBUS), USB1.2 (VBUS)
- net at SW1.2: now also R3.2, U2.24 (PC1/~RESET); no longer R1.2
- net at MX1.2 (ROW): now also D1.2 (A)
- net at MX2.2 (ROW): now also D2.2 (A)
- net at MX3.2 (ROW): now also D3.2 (A)
- net at MX10.2 (ROW): now also D10.2 (A)
- net at MX12.2 (ROW): now also D12.2 (A)
- net at MX13.2 (ROW): now also D13.2 (A)
- net at MX11.2 (ROW): now also D11.2 (A)
- new net: D22.2 (A), MX22.2 (ROW)
- new net: D21.2 (A), MX21.2 (ROW)
- new net: D20.2 (A), MX20.2 (ROW)
- new net: D33.2 (A), MX33.2 (ROW)
- new net: D32.2 (A), MX32.2 (ROW)
- new net: D31.2 (A), MX31.2 (ROW)
- new net: D30.2 (A), MX30.2 (ROW)
- new net: D42.2 (A), MX42.2 (ROW)
- new net: D40.2 (A), MX40.2 (ROW)
- new net: D0.2 (A), MX0.2 (ROW)
- new net: R1.1, USB1.10 (CC2)
- new net: R2.1, USB1.4 (CC1)
- new net: C4.1, U2.1 (XTAL1), Y1.1
- new net: R6.2, U2.13 (~HWB~/PD7)
- new net: C5.1, U2.2 (PC0/XTAL2), Y1.3
- new net: C6.1, U2.27 (UCAP)
- new net MCU_D+: R4.1, U2.29 (D+)
- new net MCU_D-: R5.1, U2.30 (D-)
- no-connect marks 20 -> 14
Other:
- note removed: "MCU Decoupling"
- note removed: "Microcontroller Interface"
- note removed: "Switch Matrix"
- note removed: "USB Interface"

Commit message: Complete PCB v1
Parts:
- removed U2: ATmega32U2-MU, Package_DFN_QFN:QFN-32-1EP_5x5mm_P0.5mm_EP3.1x3.1mm, symbol MCU_Microchip_ATmega:ATmega32U2-MU
- removed USB1: HRO-TYPE-C-31-M-12, Type-C:HRO-TYPE-C-31-M-12, symbol Type-C:HRO-TYPE-C-31-M-12
- added C7: 100nF, Capacitor_SMD:C_0603_1608Metric, symbol Device:C_Small
- added D1: D_Small, Diode_SMD:D_SOD-123, symbol Device:D_Small
- added J1: AVR-ISP-6, Connector_PinHeader_2.54mm:PinHeader_2x03_P2.54mm_Vertical, symbol Connector:AVR-ISP-6
- added R7: 330R, Resistor_SMD:R_0603_1608Metric, symbol Device:R_Small
- added U2: ATmega32U2-AU, Package_QFP:TQFP-32_7x7mm_P0.8mm, symbol MCU_Microchip_ATmega:ATmega32U2-AU
- added USB1: DX07S016JA1R1500, DX07S016JA1R1500:JAE_DX07S016JA1R1500, symbol DX07S016JA1R1500:DX07S016JA1R1500
- C1, C2, C4, C5, C6: footprint Capacitor_SMD:C_0402_1005Metric -> Capacitor_SMD:C_0603_1608Metric
- R1, R2, R3, R4, R5, R6: footprint Resistor_SMD:R_0402_1005Metric -> Resistor_SMD:R_0603_1608Metric
- renumbered D0 to D00, D1 to D01, D2 to D02, D3 to D03, MX0 to MX00, MX1 to MX01, MX2 to MX02, MX3 to MX03
Connections:
- net +5V: now also D1.1 (K), J1.2 (VCC), U2.31 (UVCC), U2.32 (AVCC), U2.4 (VCC)
- net COL0: now also U2.23 (PC6)
- net COL1: now also U2.8 (PD2)
- net COL2: now also U2.7 (PD1)
- net COL3: now also U2.6 (PD0)
- net GND: now also C7.2, J1.6 (GND), U2.28 (UGND), U2.3 (GND), USB1.1 (GND), USB1.12 (GND)
- net MCU_D+: now also U2.29 (D+)
- net MCU_D-: now also U2.30 (D-)
- net ROW0: now also U2.25 (PC5)
- net ROW1: now also U2.12 (PD6)
- net ROW2: now also U2.11 (PD5)
- net ROW3: now also U2.10 (PD4)
- net ROW4: now also U2.9 (PD3)
- net USB_D+: now also USB1.6 (D+), USB1.7 (D+)
- net USB_D-: now also USB1.5 (D-), USB1.8 (D-)
- net VCC: now also USB1.11 (VBUS), USB1.2 (VBUS)
- net at R1.1: now also USB1.9 (CC2)
- net at R2.1: now also USB1.3 (CC1)
- net at C4.1, Y1.1: now also U2.1 (XTAL1)
- net at R6.2: now also U2.13 (~HWB~/PD7)
- net at C5.1, Y1.3: now also U2.2 (PC0/XTAL2)
- net at SW1.2: now also R7.2; no longer R3.2
- net at C6.1: now also U2.27 (UCAP)
- new net: USB1.S1 (SHIELD), USB1.S2 (SHIELD), USB1.S3 (SHIELD), USB1.S4 (SHIELD), USB1.S5 (SHIELD), USB1.S6 (SHIELD)
- new net MISO: J1.1 (MISO), U2.17 (PB3)
- new net MOSI: J1.4 (MOSI), U2.16 (PB2)
- new net RESET: C7.1, D1.2 (A), J1.5 (~RST), R3.2, R7.1, U2.24 (PC1/~RESET)
- new net SCK: J1.3 (SCK), U2.15 (PB1)
- no-connect marks 14 -> 11
Other:
- note added: "1.0"
- note added: "24 Oct 2020"
- note added: "Decoupling"
- note added: "ICSP"
- note added: "Keyboard Matrix"
- note added: "Microcontroller"
- note added: "Numpad"
- note added: "Numpad Schematic"
- note added: "USB"
- note added: "USB Protection"
- moved on the sheet: C1, C2, C3, C4, C5, C6, D00, D01, D02, D03, D10, D11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
